File: STM32.sch (EAGLE design)
At the start: 35 parts, among them Q1 8MHz

Commit message: V1.0
Se termina el primer ruteado
Parts:
- removed QG1: SG-615PCG, crystal:SG-615PCG
- added Q3: MC-306, crystal:MC-306
- C12, C13, C14, C15: value 104 -> 20p
Connections:
- removed net 5V: SV4.3
- removed net N$4: C12.2, C13.2
- removed net NRST: SV3.17
- removed net SWDCLK: SV2.3
- removed net SWDIO: SV2.2
- net +3V3: no longer QG1.VCC
- net +5V: now also SV4.3
- net GND: now also C12.2, C13.2; no longer QG1.GND
- net OSC32IN: now also Q3.2; no longer QG1.FO
- net OSC32OUT: now also Q3.1; no longer QG1.OE
- net RESET: now also SV3.17
- net SWCLK: now also SV2.3
- net SWIO: now also SV2.2
Other:
- note removed: "El oscilador de 32 aún no está definido correctamente"
- moved on the sheet: C14, C15
